Commit message: Done_arm_camera_bot

File: description/robot_core.xacro (robot description, xacro)
@@ -14,10 +14,16 @@
         <color rgba="0 0 0 1"/>
     </material>
+s
+    <material name="green">
+        <color rgba="0 1 0 1" />
+    </material>
+    <material name="red">
+        <color rgba="1 0 0 1" />
+    </material>
     <!-- WORLD LINK-->
-    <link name="world_link">
-    </link>
+    <link name="world"></link>
     <!-- BASE JOINT-->
     <joint name="base_joint" type="fixed">
-        <parent link="world_link"/>
+        <parent link="world"/>
         <child link="base_link"/>
         <origin xyz="1.5 1 0" rpy="0 0 0"/>
@@ -30,5 +36,5 @@
                 <box size="2.5 1.5 0.1"/>
             </geometry>
-            <material name="blue"/>
+            <material name="green"/>
         </visual>
         <collision>
@@ -49,4 +55,5 @@
         <limit lower="0" upper="2" velocity="100" effort="100"/>
         <axis xyz="1 0 0"/>
+        <dynamics damping="10.0" friction="10.0"/>
     </joint>
     <!-- SLIDER LINK-->
@@ -57,5 +64,5 @@
             </geometry>
             <origin xyz="0 0 0.075"/>
-            <material name="black"/>
+            <material name="blue"/>
         </visual>
         <collision>
@@ -76,4 +83,5 @@
         <limit lower="0" upper="${pi/2}" velocity="100" effort="100"/>
         <axis xyz="0 -1 0"/>
+        <dynamics damping="10.0" friction="10.0"/>
     </joint>
     <!-- ARM LINK-->
@@ -130,3 +138,4 @@
         </xacro:inertial_box>
     </link>
+    <xacro:include filename="example_gazebo.xacro" />
 </robot>
